File: Hardware/Qwiic PHT Sensor - MS8607.brd (EAGLE design)
At the start: 25.4 x 25.4 mm, 36 parts, among them J3 PTH, U1 MS8607-02BA01

Commit message: Added the restrict area between the MS8607 pins
Parts:
- C1: value 0.1uF -> 0.22uF
Routing:
- net GND: vias 13 -> 15
Changed lines of the file:
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@@
 <element name="FRAME1" library="SparkFun-Aesthetics" package="CREATIVE_COMMONS" value="FRAME-LETTER" x="-20.32" y="-17.78" smashed="yes"/>
 <element name="U$2" library="SparkX" package="SPARKX-MEDIUM" value="SPARKX-LOGO4" x="12.7" y="23.495" smashed="yes" rot="MR0"/>
-<element name="C1" library="SparkFun-Capacitors" package="0603" value="0.1uF" x="12.7" y="9.525" smashed="yes">
+<element name="C1" library="SparkFun-Capacitors" library_urn="urn:adsk.eagle:library:510" package="0603" package3d_urn="urn:adsk.eagle:package:37414/1" value="0.22uF" x="12.7" y="9.525" smashed="yes">
 <attribute name="NAME" x="12.7" y="8.0645" size="0.6096" layer="25" font="vector" ratio="20" align="bottom-center"/>
-<attribute name="PROD_ID" value="CAP-00810" x="12.7" y="9.525" size="1.778" layer="27" font="vector" ratio="15" display="off"/>
+<attribute name="PROD_ID" value="CAP-07822" x="12.7" y="9.525" size="1.778" layer="27" font="vector" ratio="15" display="off"/>
 </element>
 <element name="J1" library="SparkFun-Connectors" package="1X04_1MM_RA" value="" x="20.32" y="12.7" smashed="yes" rot="R90">
@@
 <via x="3.81" y="8.89" extent="1-16" drill="0.3"/>
 <via x="15.875" y="18.0975" extent="1-16" drill="0.3"/>
+<via x="6.985" y="10.795" extent="1-16" drill="0.3"/>
+<via x="18.415" y="14.605" extent="1-16" drill="0.3"/>
 </signal>
 <signal name="SCL">
